Commit message: Work on movement and use in simulations

File: simulation/urdf/robot-simple.urdf (robot description, URDF)
Before this commit: robot legsimple, 25 links, 24 joints
Links:
- link bl_foot: mass 0.0005 -> 0.005
- link bl_hip: mass 0.02 -> 0.2
- link br_foot: mass 0.0005 -> 0.005
- link br_hip: mass 0.02 -> 0.2
- link fl_foot: mass 0.0005 -> 0.005
- link fl_hip: mass 0.02 -> 0.2
- link fr_foot: mass 0.0005 -> 0.005
- link fr_hip: mass 0.02 -> 0.2

Commit message: Continued work on simulated motion

File: simulation/urdf/robot-simple.urdf (robot description, URDF)
Before this commit: robot legsimple, 25 links, 24 joints
Links:
- link bl_foot: mass 0.005 -> 0.001
- link br_foot: mass 0.005 -> 0.001
- link fl_foot: mass 0.005 -> 0.001
- link fr_foot: mass 0.005 -> 0.001
